File: pcb/sdram-demo/sdram.kicad_sch (KiCad schematic)
At the start: 19 parts, among them U1 74HC595, U2 74HC595, U3 74HC595, U4 MT48LC16M16A2P, U5 Pico

Commit message: Update pcb
Connections:
- net SER1: now also U5.26 (GPIO20); no longer U5.21 (GPIO16)
- net SER3: now also U5.27 (GPIO21); no longer U5.31 (GPIO26_ADC0)
- net SRCLK: now also U5.30 (RUN); no longer U5.27 (GPIO21)
Changed lines of the file:
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@@
+	(wire
+		(pts
+			(xy 358.14 144.78) (xy 332.74 144.78)
+		)
+		(stroke
+			(width 0)
+			(type default)
+		)
+	)
 	(wire
 		(pts
@@
 	(wire
 		(pts
-			(xy 334.01 157.48) (xy 332.74 157.48)
-		)
-		(stroke
-			(width 0)
-			(type default)
-		)
-	)
-	(wire
-		(pts
 			(xy 297.18 144.78) (xy 269.24 144.78)
 		)
@@
 	(wire
 		(pts
-			(xy 332.74 142.24) (xy 334.01 142.24)
-		)
-		(stroke
-			(width 0)
-			(type default)
-		)
-	)
-	(wire
-		(pts
 			(xy 297.18 114.3) (xy 294.64 114.3)
 		)
@@
 	(wire
 		(pts
+			(xy 358.14 142.24) (xy 332.74 142.24)
+		)
+		(stroke
+			(width 0)
+			(type default)
+		)
+	)
+	(wire
+		(pts
 			(xy 142.24 139.7) (xy 215.9 139.7)
 		)
@@
 	(wire
 		(pts
-			(xy 334.01 132.08) (xy 332.74 132.08)
-		)
-		(stroke
-			(width 0)
-			(type default)
-		)
-	)
-	(wire
-		(pts
 			(xy 276.86 134.62) (xy 297.18 134.62)
 		)
@@
 	(wire
 		(pts
-			(xy 334.01 149.86) (xy 332.74 149.86)
+			(xy 358.14 149.86) (xy 332.74 149.86)
 		)
 		(stroke
@@
 	(wire
 		(pts
+			(xy 332.74 134.62) (xy 358.14 134.62)
+		)
+		(stroke
+			(width 0)
+			(type default)
+		)
+	)
+	(wire
+		(pts
 			(xy 297.18 127) (xy 294.64 127)
 		)
@@
 	(wire
 		(pts
-			(xy 334.01 147.32) (xy 332.74 147.32)
+			(xy 358.14 147.32) (xy 332.74 147.32)
 		)
 		(stroke
@@
 	)
 	(label "SER2"
-		(at 334.01 147.32 0)
+		(at 358.14 147.32 0)
 		(fields_autoplaced yes)
 		(effects
@@
 		)
 	)
-	(label "SRCLK"
-		(at 334.01 142.24 0)
-		(fields_autoplaced yes)
-		(effects
-			(font
-				(size 1.27 1.27)
-			)
-			(justify left bottom)
-		)
-	)
 	(label "RCLK"
 		(at 97.79 90.17 90)
@@
 		)
 	)
-	(label "SER1"
-		(at 334.01 157.48 0)
+	(label "SER3"
+		(at 358.14 142.24 0)
+		(fields_autoplaced yes)
+		(effects
+			(font
+				(size 1.27 1.27)
+			)
+			(justify left bottom)
+		)
+	)
+	(label "SRCLK"
+		(at 358.14 134.62 0)
 		(fields_autoplaced yes)
 		(effects
@@
 		)
 	)
-	(label "SER3"
-		(at 334.01 132.08 0)
+	(label "SER1"
+		(at 358.14 144.78 0)
 		(fields_autoplaced yes)
 		(effects
@@
 	)
 	(label "RCLK"
-		(at 334.01 149.86 0)
+		(at 358.14 149.86 0)
 		(fields_autoplaced yes)
 		(effects

Commit message: Update pcb and add pio code
Connections:
- net SRCLK: now also U5.22 (GPIO17); no longer U5.30 (RUN)
Changed lines of the file:
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@@
+	(wire
+		(pts
+			(xy 332.74 154.94) (xy 358.14 154.94)
+		)
+		(stroke
+			(width 0)
+			(type default)
+		)
+	)
 	(wire
 		(pts
@@
 		(pts
 			(xy 133.35 62.23) (xy 133.35 59.69)
-		)
-		(stroke
-			(width 0)
-			(type default)
-		)
-	)
-	(wire
-		(pts
-			(xy 332.74 134.62) (xy 358.14 134.62)
 		)
 		(stroke
@@
 		)
 	)
+	(label "SRCLK"
+		(at 358.14 154.94 0)
+		(fields_autoplaced yes)
+		(effects
+			(font
+				(size 1.27 1.27)
+			)
+			(justify left bottom)
+		)
+	)
 	(label "SER2"
 		(at 91.44 168.91 180)
@@
 		(fields_autoplaced yes)
 		(effects
-			(font
-				(size 1.27 1.27)
-			)
-			(justify left bottom)
-		)
-	)
-	(label "SRCLK"
-		(at 358.14 134.62 0)
-		(fields_autoplaced yes)
-		(effects
