File: pcb/sdram-demo/sdram.kicad_sch (KiCad schematic)
At the start: 19 parts, among them U1 74HC595, U2 74HC595, U3 74HC595, U4 MT48LC16M16A2P, U5 Pico

Commit message: Add rev2 PCB
Parts:
- removed C1, C10, C11, C12, C4, C6, C7, C8, C9: 100n, Capacitor_SMD:C_0805_2012Metric_Pad1.18x1.45mm_HandSolder, symbol Device:C
- removed C3: 2.2u, Capacitor_SMD:C_0805_2012Metric_Pad1.18x1.45mm_HandSolder, symbol Device:C
- added JP1: Jumper_2_Open, Jumper:SolderJumper-2_P1.3mm_Open_Pad1.0x1.5mm, symbol Jumper:Jumper_2_Open
- U1, U2, U3: footprint Package_SO:TSSOP-16_4.4x5mm_P0.65mm -> Package_SO:SOIC-16_3.9x9.9mm_P1.27mm
- renumbered C5 to C1, C13 to C3, C14 to C4
Connections:
- net at U3.1 (QB): now also U4.15 (DQML); no longer U4.39 (DQMH)
- net at U3.15 (QA): no longer U4.15 (DQML)
- net at U3.2 (QC): now also U4.16 (~{WE}); no longer U4.37 (CKE)
- net at U4.19 (~{CS}): now also U5.31 (GPIO26_ADC0), JP1.2 (B); no longer U3.3 (QD)
- net at U4.17 (~{CAS}): now also U3.3 (QD); no longer U3.5 (QF)
- net at U3.6 (QG): now also U4.39 (DQMH); no longer U4.16 (~{WE})
- net at U2.1 (QB): now also JP1.1 (A)
- new net: U3.5 (QF), U4.37 (CKE)
