File: pcb/sdram-demo/sdram.kicad_pcb (KiCad board)
At the start: 2 copper layers, 25 x 55 mm, 19 parts, among them U1 74HC595, U2 74HC595, U3 74HC595, U4 MT48LC16M16A2P, U5 Pico

Commit message: Add two tests
Routing:
- net GND: vias 10 -> 16
Changed lines of the file:
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@@
+	)
+	(via
+		(at 27.5 26.5)
+		(size 0.6)
+		(drill 0.3)
+		(layers "F.Cu" "B.Cu")
+		(free yes)
+		(net 2)
 	)
 	(via
@@
 	)
 	(via
+		(at 37.5 23)
+		(size 0.6)
+		(drill 0.3)
+		(layers "F.Cu" "B.Cu")
+		(free yes)
+		(net 2)
+	)
+	(via
 		(at 30.710996 40.43)
+		(size 0.6)
+		(drill 0.3)
+		(layers "F.Cu" "B.Cu")
+		(free yes)
+		(net 2)
+	)
+	(via
+		(at 27.5 24.5)
+		(size 0.6)
+		(drill 0.3)
+		(layers "F.Cu" "B.Cu")
+		(free yes)
+		(net 2)
+	)
+	(via
+		(at 38.5 23)
 		(size 0.6)
 		(drill 0.3)
@@
 	)
 	(via
+		(at 27.5 25.5)
+		(size 0.6)
+		(drill 0.3)
+		(layers "F.Cu" "B.Cu")
+		(free yes)
+		(net 2)
+	)
+	(via
 		(at 39.710996 43.33)
 		(size 0.6)
@@
 		(size 0.6)
 		(drill 0.3)
+		(layers "F.Cu" "B.Cu")
+		(free yes)
+		(net 2)
+	)
+	(via
+		(at 39.5 23)
+		(size 0.6)
+		(drill 0.3)

Commit message: wip - adding input mode on data bus
Other:
- board text added: "Pico SDRAM Shield - Rev 1 - Ethan James 2024"
Changed lines of the file:
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@@
 		(layer "Edge.Cuts")
+	)
+	(gr_text "Pico SDRAM Shield - Rev 1 - Ethan James 2024"
+		(at 43.4 75.7 270)
+		(layer "B.SilkS")
+		(effects
+			(font
+				(size 1 1)
+				(thickness 0.1)
+			)
+			(justify left bottom mirror)
+		)
 	)
 	(segment

Commit message: Add rev2 PCB
Parts:
- removed C10, C11, C12, C13, C6, C7, C8, C9: 100n, Capacitor_SMD:C_0805_2012Metric_Pad1.18x1.45mm_HandSolder
- removed C14, C5: 2.2u, Capacitor_SMD:C_0805_2012Metric_Pad1.18x1.45mm_HandSolder
- added JP1: Jumper_2_Open, Jumper:SolderJumper-2_P1.3mm_Open_Pad1.0x1.5mm, B.Cu at (156.3, 124.9)
- C1, C4: value 100n -> 2.2u
- C3: value 2.2u -> 100n
- U1, U2, U3: footprint Package_SO:TSSOP-16_4.4x5mm_P0.65mm -> Package_SO:SOIC-16_3.9x9.9mm_P1.27mm
- moved U1 129.0 mm to (146.6, 118.3)
- moved U2 128.9 mm to (154.5, 118.3)
- moved U5 128.7 mm to (150.6, 100.8)
- moved U3 128.4 mm to (150.5, 84.9), turned to 90 degrees
- moved U4 128.3 mm to (150.6, 100.5)
- moved C3 121.7 mm to (156.4, 76.8)
- moved C1 117.9 mm to (144.6, 76.8)
- moved C4 117.7 mm to (156.0, 79.0), turned to 180 degrees
- moved C2 114.7 mm to (145.0, 79.0), turned to 180 degrees
Connections:
- U2 pad 1: unconnected-(U2-QB-Pad1) -> Net-(JP1-A)
- U3 pad 15: Net-(U3-QA) -> unconnected-(U3-QA-Pad15)
- U4 pad 15: Net-(U3-QA) -> Net-(U3-QB)
- U4 pad 16: Net-(U3-QG) -> Net-(U3-QC)
- U4 pad 17: Net-(U3-QF) -> Net-(U3-QD)
- U4 pad 19: Net-(U3-QD) -> Net-(JP1-B)
- U4 pad 37: Net-(U3-QC) -> Net-(U3-QF)
- U4 pad 39: Net-(U3-QB) -> Net-(U3-QG)
- U5 pad 31: unconnected-(U5-GPIO26_ADC0-Pad31) -> Net-(JP1-B)
Routing:
- net Net-(JP1-B): track 0.00 -> 35.7 mm
- net Net-(JP1-A): track 0.00 -> 18.7 mm
- net Net-(U3-QA): track 18.4 -> 0.00 mm
- net +3V3: track 152.9 -> 135.6 mm, vias 12 -> 2
- net Net-(U3-QC): track 24.6 -> 17.4 mm
- net Net-(U3-QD): track 23.8 -> 17.8 mm
- net Net-(U3-QG): track 23.3 -> 17.7 mm
- net Net-(U3-QB): track 21.8 -> 16.9 mm
- net Net-(U3-QE): track 23.6 -> 19.0 mm
- net /SER3: track 39.8 -> 36.2 mm
- net Net-(U3-QF): track 23.5 -> 20.0 mm, vias 0 -> 2
- net Net-(U2-QH): track 16.1 -> 18.9 mm
- net Net-(U4-DQ6): track 26.5 -> 24.0 mm
- net Net-(U4-DQ7): track 29.6 -> 27.1 mm
- net Net-(U4-DQ5): track 21.6 -> 19.1 mm
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Other:
- board text added: "Pico SDRAM Shield - Rev 2 - Ethan James 2024"
- board text removed: "Pico SDRAM Shield - Rev 1 - Ethan James 2024"
